Commit message: Completed Task A.4, A.5, and A.6 Still having issues with color of robots in rviz

File: nuturtle_description/urdf/colors.urdf.xacro (robot description, xacro)
@@ -7,5 +7,5 @@
     </material>
     <material name="purple">
-        <color rgba="0.3 0.16 0.0.52 1"/>
+        <color rgba="0.3 0.16 0.52 1"/>
     </material>
     <material name="blue">

File: nuturtle_description/urdf/turtlebot3_burger.urdf.xacro (robot description, xacro)
@@ -4,9 +4,10 @@
   <!-- <xacro:include filename="$(find turtlebot3_description)/urdf/common_properties.urdf"/> -->
   <xacro:property name="turtlebot_config" value="${xacro.load_yaml('$(find nuturtle_description)/config/diff_params.yaml')}"/>
-  <xacro:include filename="materials.urdf.xacro"/>
+  <xacro:include filename="colors.urdf.xacro"/>
   <xacro:property name="wheel_radius" value="${turtlebot_config['/**']['ros__parameters']['wheel_radius']}"/>
-  <xacro:property name="track_width" value="${turtle_config['/**']['ros__parameters']['track_width']}"/>
-  <xacro:property name="collision_radius" value="${turtle_config['/**']['ros__parameters']['collision_radius']}"/>
+  <xacro:property name="track_width" value="${turtlebot_config['/**']['ros__parameters']['track_width']}"/>
+  <xacro:property name="collision_radius" value="${turtlebot_config['/**']['ros__parameters']['collision_radius']}"/>
   <xacro:arg name="color" default="purple"/>
+  <xacro:property name="color" value="$(arg color)"/>
   <xacro:arg name="namespace" default=""/>
   <xacro:property name="namespace" value="$(arg namespace)"/>
@@ -21,10 +22,4 @@
     <color rgba="0.4 0.4 0.4 1.0"/>
   </material>
-  <material name="blue">
-    <color rgba="0.0 0.0 0.8 1.0"/>
-  </material>
-  <material name="green">
-    <color rgba="0.0 0.8 0.0 1.0"/>
-  </material>
   <material name="grey">
     <color rgba="0.5 0.5 0.5 1.0"/>
@@ -35,7 +30,4 @@
   <material name="brown">
     <color rgba="0.8706 0.8118 0.7647 1.0"/>
-  </material>
-  <material name="red">
-    <color rgba="0.8 0.0 0.0 1.0"/>
   </material>
   <material name="white">
@@ -52,5 +44,5 @@
       <origin xyz="-0.032 0 0.0" rpy="0 0 0"/>
       <geometry>
-        <mesh filename="package://nuturtle_description/meshes/bases/burger_base.stl" scale="0.001 0.001 0.001"/>
+        <mesh filename="package://nuturtle_description/mesh/burger_base.stl" scale="0.001 0.001 0.001"/>
       </geometry>
       <material name="${color}"/>
@@ -71,5 +63,5 @@
     <parent link="${namespace}base_link"/>
     <child link="${namespace}wheel_left_link"/>
-    <origin xyz="0.0 ${track_width}/2 0.023" rpy="-1.57 0 0"/>
+    <origin xyz="0.0 ${track_width/2} 0.023" rpy="-1.57 0 0"/>
     <axis xyz="0 0 1"/>
   </joint>
@@ -78,5 +70,5 @@
       <origin xyz="0 0 0" rpy="1.57 0 0"/>
       <geometry>
-        <mesh filename="package://nuturtle_description/meshes/wheels/left_tire.stl" scale="0.001 0.001 0.001"/>
+        <mesh filename="package://nuturtle_description/mesh/wheels/left_tire.stl" scale="0.001 0.001 0.001"/>
       </geometry>
       <material name="dark"/>
@@ -97,5 +89,5 @@
     <parent link="${namespace}base_link"/>
     <child link="${namespace}wheel_right_link"/>
-    <origin xyz="0.0 -${track_width}/2 0.023" rpy="-1.57 0 0"/>
+    <origin xyz="0.0 -${track_width/2} 0.023" rpy="-1.57 0 0"/>
     <axis xyz="0 0 1"/>
   </joint>
@@ -104,5 +96,5 @@
       <origin xyz="0 0 0" rpy="1.57 0 0"/>
       <geometry>
-        <mesh filename="package://nuturtle_description/meshes/wheels/right_tire.stl" scale="0.001 0.001 0.001"/>
+        <mesh filename="package://nuturtle_description/mesh/wheels/right_tire.stl" scale="0.001 0.001 0.001"/>
       </geometry>
       <material name="dark"/>
@@ -153,5 +145,5 @@
       <origin xyz="0 0 0.0" rpy="0 0 0"/>
       <geometry>
-        <mesh filename="package://nuturtle_description/meshes/sensors/lds.stl" scale="0.001 0.001 0.001"/>
+        <mesh filename="package://nuturtle_description/mesh/lds.stl" scale="0.001 0.001 0.001"/>
       </geometry>
       <material name="dark"/>
